File: Palm Vein Illuminator.kicad_pcb (KiCad board)
At the start: 2 copper layers, 0 parts

Commit message: Add PCB component placement
Parts:
- added C1: CL21B105KBFNNNE, JLCImport:CL21B105KBFNNNE, F.Cu at (197.5, 61.5)
- added C10: CL05B104KO5NNNC, JLCImport:CL05B104KO5NNNC, F.Cu at (192.5, 108.1)
- added C11: TAJA226K010RNJ, JLCImport:TAJA226K010RNJ, F.Cu at (214.5, 87.3)
- added C12: CC0805MKX7R7BB106, JLCImport:CC0805MKX7R7BB106, F.Cu at (210.5, 87.3)
- added C13: CL05B104KO5NNNC, JLCImport:CL05B104KO5NNNC, F.Cu at (207.5, 81.8)
- added C14: CL05B104KO5NNNC, JLCImport:CL05B104KO5NNNC, F.Cu at (196.4, 94.0)
- added C15: CL21B475KOFNNNE, JLCImport:CL21B475KOFNNNE, F.Cu at (196.3, 96.0)
- added C2: CL05B104KB54PNC, JLCImport:CL05B104KB54PNC, F.Cu at (197.5, 52.5)
- added C3: 0603B222K500NT, JLCImport:0603B222K500NT, F.Cu at (205.0, 53.7)
- added C4: RVT1H331M1010, JLCImport:RVT1H331M1010, B.Cu at (195.7, 54.5)
- added C5: CS3225X7R106K500NRL, JLCImport:CS3225X7R106K500NRL, F.Cu at (192.4, 58.0)
- added C6: CS3225X7R106K500NRL, JLCImport:CS3225X7R106K500NRL, F.Cu at (192.4, 69.5)
- added C7: HGC1210R5107M160NSVK, JLCImport:HGC1210R5107M160NSVK, F.Cu at (208.6, 109.5)
- added C8: CS3225X7R106K500NRL, JLCImport:CS3225X7R106K500NRL, F.Cu at (186.0, 105.1)
- added C9: CL31B225KBHNNNE, JLCImport:CL31B225KBHNNNE, F.Cu at (186.3, 108.0)
- added D1: TDS2211P.C(ES), JLCImport:TDS2211P.C(ES), F.Cu at (196.7, 49.7)
- added D10: SFH_4718A, JLCImport:SFH_4718A, F.Cu at (170.0, 116.2)
- added D11: SS34_C8678, JLCImport:SS34_C8678, F.Cu at (192.6, 65.5)
- added D12: SFH_4718A, JLCImport:SFH_4718A, F.Cu at (170.0, 59.6)
- added D13: SFH_4718A, JLCImport:SFH_4718A, F.Cu at (170.0, 73.8)
- added D14: SFH_4718A, JLCImport:SFH_4718A, F.Cu at (170.0, 87.9)
- added D15: SFH_4718A, JLCImport:SFH_4718A, F.Cu at (170.0, 102.1)
- added D16: SFH_4718A, JLCImport:SFH_4718A, F.Cu at (220.7, 102.1)
- added D17: SFH_4718A, JLCImport:SFH_4718A, F.Cu at (220.7, 87.9)
- added D18: SFH_4718A, JLCImport:SFH_4718A, F.Cu at (220.7, 73.8)
- added D19: SFH_4718A, JLCImport:SFH_4718A, F.Cu at (220.7, 59.6)
- added D2: SS34_C8678, JLCImport:SS34_C8678, F.Cu at (192.6, 54.0)
- added D3: SFH_4718A, JLCImport:SFH_4718A, F.Cu at (170.0, 45.5)
- added D4: SFH_4718A, JLCImport:SFH_4718A, F.Cu at (185.8, 45.5)
- added D5: SFH_4718A, JLCImport:SFH_4718A, F.Cu at (203.8, 45.5)
- added D6: SFH_4718A, JLCImport:SFH_4718A, F.Cu at (220.7, 45.5)
- added D7: SFH_4718A, JLCImport:SFH_4718A, F.Cu at (220.7, 116.2)
- added D8: SFH_4718A, JLCImport:SFH_4718A, F.Cu at (203.8, 116.2)
- added D9: SFH_4718A, JLCImport:SFH_4718A, F.Cu at (185.8, 116.2)
- added H1: MountingHole_2.2mm_M2, MountingHole:MountingHole_2.2mm_M2, F.Cu at (170.0, 52.6)
- added H2: MountingHole_2.2mm_M2, MountingHole:MountingHole_2.2mm_M2, F.Cu at (220.7, 52.6)
- added H3: MountingHole_2.2mm_M2, MountingHole:MountingHole_2.2mm_M2, F.Cu at (170.0, 109.1)
- added H4: MountingHole_2.2mm_M2, MountingHole:MountingHole_2.2mm_M2, F.Cu at (220.7, 109.1)
- added H5: MountingHole_2.2mm_M2, MountingHole:MountingHole_2.2mm_M2, F.Cu at (185.2, 75.6)
- added H6: MountingHole_2.2mm_M2, MountingHole:MountingHole_2.2mm_M2, F.Cu at (206.2, 75.6)
- added H7: MountingHole_2.2mm_M2, MountingHole:MountingHole_2.2mm_M2, F.Cu at (185.2, 88.1)
- added H8: MountingHole_2.2mm_M2, MountingHole:MountingHole_2.2mm_M2, F.Cu at (206.2, 88.1)
- added J1: TYPE-C-31-M-12, JLCImport:TYPE-C-31-M-12, F.Cu at (194.8, 45.0)
- added J2: S6P-VH_LF_SN, JLCImport:S6P-VH_LF_SN, B.Cu at (195.5, 98.9)
- added J3: PZ2_54-1X4PWZ-L13_8-A, JLCImport:PZ2_54-1X4PWZ-L13_8-A, B.Cu at (211.5, 68.0)
- added L1: NRSE8040-470M, JLCImport:NRSE8040-470M, F.Cu at (179.0, 56.5)
- added L2: NRSE8040-470M, JLCImport:NRSE8040-470M, F.Cu at (179.0, 68.0)
- added L3: PNLS8040-2R2, JLCImport:PNLS8040-2R2, F.Cu at (200.5, 107.0)
- added R1: 0603WAF1203T5E, JLCImport:0603WAF1203T5E, F.Cu at (208.3, 61.2)
- added R10: 0603WAF1003T5E, JLCImport:0603WAF1003T5E, F.Cu at (186.3, 102.6)
- added R11: 0603WAF3601T5E, JLCImport:0603WAF3601T5E, F.Cu at (191.6, 90.5)
- added R12: 0603WAF1002T5E, JLCImport:0603WAF1002T5E, F.Cu at (191.6, 92.5)
- added R13: 0603WAF1002T5E, JLCImport:0603WAF1002T5E, F.Cu at (191.6, 94.5)
- added R14: 0603WAF3601T5E, JLCImport:0603WAF3601T5E, F.Cu at (191.6, 96.5)
- added R2: 0603WAF1003T5E, JLCImport:0603WAF1003T5E, F.Cu at (209.6, 50.5)
- added R3: 0603WAF2701T5E, JLCImport:0603WAF2701T5E, F.Cu at (209.6, 52.5)
- added R4: 0603WAF6201T5E, JLCImport:0603WAF6201T5E, F.Cu at (209.6, 54.5)
- added R5: 0603WAF4301T5E, JLCImport:0603WAF4301T5E, F.Cu at (209.6, 56.5)
- added R6: RLH12FTCR110, JLCImport:RLH12FTCR110, F.Cu at (186.5, 53.5)
- added R7: RLH12FTCR110, JLCImport:RLH12FTCR110, F.Cu at (186.5, 65.0)
- added R8: 0603WAF2203T5E, JLCImport:0603WAF2203T5E, F.Cu at (184.3, 110.1)
- added R9: 0603WAF3002T5E, JLCImport:0603WAF3002T5E, F.Cu at (187.3, 110.1)
- added U1: CH224A, JLCImport:CH224A, F.Cu at (203.0, 62.0)
- added U2: MX25947ES, JLCImport:MX25947ES, F.Cu at (201.1, 53.5)
- added U3: AL8861Y-13, JLCImport:AL8861Y-13, F.Cu at (186.6, 57.5)
- added U4: AL8861Y-13, JLCImport:AL8861Y-13, F.Cu at (186.6, 69.0)
- added U5: SY8366HQQC, JLCImport:SY8366HQQC, F.Cu at (190.9, 105.2)
- added U6: AMS1117-3_3_C347222, JLCImport:AMS1117-3_3_C347222, F.Cu at (212.5, 94.1)
- added U7: CH32V003A4M6, JLCImport:CH32V003A4M6, F.Cu at (212.5, 79.5)
- added U8: VL53L4CDV0DH_1, JLCImport:VL53L4CDV0DH_1, F.Cu at (195.7, 92.1)
Other:
- board outline added: 59.7 x 79.7 mm

Commit message: Route PCB and add copper pours
Routing:
- net +20V: track 0.00 -> 119.5 mm, vias 0 -> 7
- net +3.3V: track 0.00 -> 93.9 mm
- net Net-(U3-ISENSE): track 0.00 -> 87.5 mm, vias 0 -> 12
- net Net-(D7--): track 0.00 -> 74.7 mm, vias 0 -> 8
- net Net-(D16--): track 0.00 -> 72.0 mm, vias 0 -> 8
- net /VHV: track 0.00 -> 63.0 mm, vias 0 -> 9
- net /DN: track 0.00 -> 57.0 mm, vias 0 -> 2
- net /DP: track 0.00 -> 56.1 mm, vias 0 -> 2
- net +5V: track 0.00 -> 50.4 mm
- net Net-(U4-ISENSE): track 0.00 -> 50.1 mm, vias 0 -> 12
- net /CC1: track 0.00 -> 45.6 mm, vias 0 -> 2
- net /SDA: track 0.00 -> 45.2 mm, vias 0 -> 2
- net Net-(U7-PD5): track 0.00 -> 45.0 mm, vias 0 -> 1
- net /PWM1: track 0.00 -> 43.6 mm, vias 0 -> 4
- net /SCL: track 0.00 -> 43.0 mm, vias 0 -> 4
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- added copper zone on B.Cu, net GND
- added copper zone on F.Cu, net GND
- added copper zone on B.Cu, net Net-(D10--)
- added copper zone on F.Cu, net Net-(D10--)
- added copper zone on B.Cu, net Net-(D13--)
- added copper zone on F.Cu, net Net-(D13--)
- added copper zone on B.Cu, net Net-(D14--)
- added copper zone on F.Cu, net Net-(D14--)
- added copper zone on B.Cu, net Net-(D15--)
- added copper zone on F.Cu, net Net-(D15--)
- added copper zone on B.Cu, net Net-(D16--)
- added copper zone on F.Cu, net Net-(D16--)
- added copper zone on B.Cu, net Net-(D17--)
- added copper zone on F.Cu, net Net-(D17--)
- added copper zone on B.Cu, net Net-(D18--)
- added copper zone on F.Cu, net Net-(D18--)
- added copper zone on B.Cu, net Net-(D19--)
- added copper zone on F.Cu, net Net-(D19--)
- added copper zone on B.Cu, net Net-(D4--)
- added copper zone on F.Cu, net Net-(D4--)
- added copper zone on B.Cu, net Net-(D5--)
- added copper zone on F.Cu, net Net-(D5--)
- added copper zone on B.Cu, net Net-(D6--)
- added copper zone on F.Cu, net Net-(D6--)
- added copper zone on B.Cu, net Net-(D7--)
- added copper zone on F.Cu, net Net-(D7--)
- added copper zone on B.Cu, net Net-(D8--)
- added copper zone on F.Cu, net Net-(D8--)
- added copper zone on B.Cu, net Net-(D9--)
- added copper zone on F.Cu, net Net-(D9--)
- added copper zone on B.Cu, net Net-(U3-ISENSE)
- added copper zone on F.Cu, net Net-(U3-ISENSE)
- added copper zone on B.Cu, net Net-(U4-ISENSE)
- added copper zone on F.Cu, net Net-(U4-ISENSE)
- added copper zone on F.Cu, net Net-(U5-LX)
